File: PSoC 4 Prototyping Kit DCO/eagle/PSoC4_Prototyping_Kit_DCO/PSoC4_Prototyping_Kit_DCO.brd (EAGLE design)
At the start: 48.2 x 73.3 mm, 13 parts, among them IC1 PSOC_4_PROTOTYPING_KIT

Commit message: Add a inverse Diode from VDD to GND
Parts:
- added D1: 1S4, diode:DO35-7
Connections:
- net +3V3: now also D1.C
- net GND: now also D1.A
Routing:
- net +3V3: track 29.0 -> 32.6 mm
- net GND: track 78.3 -> 80.8 mm
Changed lines of the file:
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@@
 <layer number="97" name="Info" color="7" fill="1" visible="no" active="no"/>
 <layer number="98" name="Guide" color="6" fill="1" visible="no" active="no"/>
+<layer number="99" name="SpiceOrder" color="5" fill="1" visible="no" active="no"/>
 <layer number="100" name="Grid" color="11" fill="1" visible="yes" active="yes"/>
 <layer number="200" name="200bmp" color="1" fill="10" visible="no" active="no"/>
@@
 <element name="JP5" library="pinhead" package="1X02" value="PWR" x="7.62" y="11.43" rot="R90"/>
 <element name="JP2" library="pinhead" package="1X04" value="SPI" x="7.62" y="39.37" rot="R90"/>
+<element name="D1" library="diode" package="DO35-7" value="1S4" x="2.54" y="11.43" rot="R90"/>
 </elements>
 <signals>
@@
 <wire x1="17.78" y1="5.08" x2="20.32" y2="7.62" width="0.4064" layer="16"/>
 <wire x1="20.32" y1="7.62" x2="20.32" y2="10.16" width="0.4064" layer="16"/>
+<contactref element="D1" pad="C"/>
+<wire x1="2.54" y1="7.62" x2="5.08" y2="10.16" width="0.4064" layer="16"/>
 </signal>
 <signal name="GND">
@@
 <wire x1="15.24" y1="33.02" x2="17.78" y2="30.48" width="0.4064" layer="16"/>
 <wire x1="20.32" y1="12.7" x2="25.4" y2="12.7" width="0.4064" layer="16"/>
-<wire x1="5.08" y1="12.7" x2="5.08" y2="17.78" width="0.4064" layer="16"/>
+<wire x1="5.08" y1="12.7" x2="5.08" y2="15.24" width="0.4064" layer="16"/>
+<wire x1="5.08" y1="15.24" x2="5.08" y2="17.78" width="0.4064" layer="16"/>
 <wire x1="5.08" y1="43.18" x2="2.54" y2="43.18" width="0.4064" layer="16"/>
 <wire x1="2.54" y1="43.18" x2="2.54" y2="30.48" width="0.4064" layer="16"/>
@@
 <wire x1="7.62" y1="12.7" x2="10.16" y2="12.7" width="0.4064" layer="16"/>
 <wire x1="10.16" y1="12.7" x2="20.32" y2="12.7" width="0.4064" layer="16"/>
+<contactref element="D1" pad="A"/>
+<wire x1="2.54" y1="15.24" x2="5.08" y2="15.24" width="0.4064" layer="16"/>
 </signal>
 <signal name="N$1">

Commit message: Add: Reset Line
Parts:
- JP1, JP2, JP3: device pinhead:1X04 -> pinhead:1X05
- moved JP1 1.27 mm to (5.08, 40.6)
- moved JP2 1.27 mm to (7.62, 40.6)
- moved JP3 1.27 mm to (10.2, 40.6)
Connections:
- new net RESET: IC1.20, JP1.5, JP2.5, JP3.5
Routing:
- net RESET: track 0.00 -> 58.2 mm
Changed lines of the file:
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@@
 <element name="IC1" library="mylib2" package="DIL44-8" value="PSOC_4_PROTOTYPING_KIT" x="38.1" y="36.83" rot="R90"/>
 <element name="JK1" library="mylib2" package="ATD_RCA_JACK_DIP" value="ATD_RCA_JACK-DIP" x="7.62" y="24.13"/>
-<element name="JP1" library="pinhead" package="1X04" value="SPI" x="5.08" y="39.37" rot="R90"/>
 <element name="JP4" library="pinhead" package="1X02" value="PWR" x="5.08" y="11.43" rot="R90"/>
 <element name="R1" library="rcl" package="0207/7" value="1k" x="19.05" y="33.02" rot="R180"/>
@@
 <element name="LED1" library="led" package="LED3MM" value="Green" x="13.97" y="5.08" rot="R180"/>
 <element name="R3" library="rcl" package="0207/7" value="1k" x="10.16" y="8.89" rot="R270"/>
-<element name="JP3" library="pinhead" package="1X04" value="SPI" x="10.16" y="39.37" rot="R90"/>
 <element name="JP5" library="pinhead" package="1X02" value="PWR" x="7.62" y="11.43" rot="R90"/>
-<element name="JP2" library="pinhead" package="1X04" value="SPI" x="7.62" y="39.37" rot="R90"/>
 <element name="D1" library="diode" package="DO35-7" value="1S4" x="2.54" y="11.43" rot="R90"/>
+<element name="JP1" library="pinhead" package="1X05" value="SPI" x="5.08" y="40.64" rot="R90"/>
+<element name="JP2" library="pinhead" package="1X05" value="SPI" x="7.62" y="40.64" rot="R90"/>
+<element name="JP3" library="pinhead" package="1X05" value="SPI" x="10.16" y="40.64" rot="R90"/>
 </elements>
 <signals>
@@
 <contactref element="C1" pad="-"/>
 <contactref element="R1" pad="2"/>
-<contactref element="JP1" pad="4"/>
 <contactref element="JK1" pad="P$5"/>
 <contactref element="JK1" pad="P$6"/>
@@
 <wire x1="5.08" y1="12.7" x2="5.08" y2="15.24" width="0.4064" layer="16"/>
 <wire x1="5.08" y1="15.24" x2="5.08" y2="17.78" width="0.4064" layer="16"/>
-<wire x1="5.08" y1="43.18" x2="2.54" y2="43.18" width="0.4064" layer="16"/>
 <wire x1="2.54" y1="43.18" x2="2.54" y2="30.48" width="0.4064" layer="16"/>
-<contactref element="JP3" pad="4"/>
 <contactref element="JP5" pad="2"/>
-<contactref element="JP2" pad="4"/>
 <contactref element="R3" pad="1"/>
-<wire x1="5.08" y1="43.18" x2="7.62" y2="43.18" width="0.4064" layer="16"/>
-<wire x1="7.62" y1="43.18" x2="10.16" y2="43.18" width="0.4064" layer="16"/>
 <wire x1="5.08" y1="12.7" x2="7.62" y2="12.7" width="0.4064" layer="16"/>
 <wire x1="7.62" y1="12.7" x2="10.16" y2="12.7" width="0.4064" layer="16"/>
@@
 <contactref element="D1" pad="A"/>
 <wire x1="2.54" y1="15.24" x2="5.08" y2="15.24" width="0.4064" layer="16"/>
+<contactref element="JP1" pad="4"/>
+<contactref element="JP2" pad="4"/>
+<contactref element="JP3" pad="4"/>
+<wire x1="2.54" y1="43.18" x2="5.08" y2="43.18" width="0.4064" layer="16"/>
+<wire x1="5.08" y1="43.18" x2="7.62" y2="43.18" width="0.4064" layer="16"/>
+<wire x1="7.62" y1="43.18" x2="10.16" y2="43.18" width="0.4064" layer="16"/>
 </signal>
 <signal name="N$1">
@@
 <signal name="MOSI">
 <contactref element="IC1" pad="31"/>
-<contactref element="JP1" pad="3"/>
 <wire x1="20.32" y1="40.64" x2="22.86" y2="43.18" width="0.4064" layer="16"/>
 <wire x1="22.86" y1="43.18" x2="25.4" y2="43.18" width="0.4064" layer="16"/>
+<contactref element="JP1" pad="3"/>
+<contactref element="JP2" pad="3"/>
 <contactref element="JP3" pad="3"/>
-<contactref element="JP2" pad="3"/>
 <wire x1="5.08" y1="40.64" x2="7.62" y2="40.64" width="0.4064" layer="16"/>
 <wire x1="7.62" y1="40.64" x2="10.16" y2="40.64" width="0.4064" layer="16"/>
@@
 <contactref element="IC1" pad="33"/>
 <contactref element="JP1" pad="2"/>
+<contactref element="JP2" pad="2"/>
 <contactref element="JP3" pad="2"/>
-<contactref element="JP2" pad="2"/>
 <wire x1="5.08" y1="38.1" x2="7.62" y2="38.1" width="0.4064" layer="16"/>
 <wire x1="7.62" y1="38.1" x2="10.16" y2="38.1" width="0.4064" layer="16"/>
@@
 <contactref element="JP2" pad="1"/>
 <contactref element="JP3" pad="1"/>
+<wire x1="10.16" y1="35.56" x2="25.4" y2="35.56" width="0.4064" layer="16"/>
 <wire x1="5.08" y1="35.56" x2="7.62" y2="35.56" width="0.4064" layer="16"/>
 <wire x1="7.62" y1="35.56" x2="10.16" y2="35.56" width="0.4064" layer="16"/>
-<wire x1="10.16" y1="35.56" x2="25.4" y2="35.56" width="0.4064" layer="16"/>
 </signal>
 <signal name="N$5">
@@
 <wire x1="10.16" y1="5.08" x2="12.7" y2="5.08" width="0.4064" layer="16"/>
 </signal>
+<signal name="RESET">
+<contactref element="IC1" pad="20"/>
+<contactref element="JP1" pad="5"/>
+<contactref element="JP2" pad="5"/>
+<contactref element="JP3" pad="5"/>
+<wire x1="5.08" y1="45.72" x2="7.62" y2="45.72" width="0.4064" layer="16"/>
+<wire x1="7.62" y1="45.72" x2="10.16" y2="45.72" width="0.4064" layer="16"/>
+<wire x1="45.72" y1="58.42" x2="43.18" y2="58.42" width="0.4064" layer="16"/>
+<wire x1="43.18" y1="58.42" x2="35.56" y2="66.04" width="0.4064" layer="16"/>
+<wire x1="35.56" y1="66.04" x2="20.32" y2="66.04" width="0.4064" layer="16"/>
+<wire x1="20.32" y1="66.04" x2="10.16" y2="55.88" width="0.4064" layer="16"/>
+<wire x1="10.16" y1="55.88" x2="10.16" y2="45.72" width="0.4064" layer="16"/>
+</signal>
 </signals>
